File: ECAD/TemperatureSensing.sch (KiCad schematic (older format))
At the start: 9 parts, among them U6 MCP6L91T-EOT, U7 MCP9700AT-ETT

Commit message: routing almost done
Parts:
- removed C19: DNP, symbol Device:C
- removed R15: 0, Resistor_SMD:R_0402_1005Metric, symbol Device:R
- removed R16: 10k, Resistor_SMD:R_0402_1005Metric, symbol Device:R
- removed U6: MCP6L91T-EOT, Package_TO_SOT_SMD:SOT-23-5, symbol Amplifier_Operational:MCP6L91T-EOT
- added C26, C29: 1n, Capacitor_SMD:C_0402_1005Metric, symbol OtterIronProRedesign-rescue:C-Device
- added C28: DNP, Capacitor_SMD:C_0402_1005Metric, symbol Device:C
- added C31: 100nF, Capacitor_SMD:C_0402_1005Metric, symbol OtterIronProRedesign-rescue:C-Device
- added JP1: Jumper, Jumper:SolderJumper-2_P1.3mm_Open_TrianglePad1.0x1.5mm, symbol Device:Jumper
- added R15, R16, R18: 22, Resistor_SMD:R_0402_1005Metric, symbol OtterIronProRedesign-rescue:R-Device
- added R19: 68k, Resistor_SMD:R_0402_1005Metric, symbol Device:R
- added R20: 560k, Resistor_SMD:R_0402_1005Metric, symbol Device:R
- added U7: TLV2376, Package_SO:SOIC-8_3.9x4.9mm_P1.27mm, symbol Device:Opamp_Dual_Generic
- C25: renamed from C21; symbol Device:C -> OtterIronProRedesign-rescue:C-Device
- C27: renamed from C20; value DNP -> 1n; footprint (none) -> Capacitor_SMD:C_0402_1005Metric; symbol Device:C -> OtterIronProRedesign-rescue:C-Device
- C30: renamed from C22; value DNP -> 1n; footprint (none) -> Capacitor_SMD:C_0402_1005Metric; symbol Device:C -> OtterIronProRedesign-rescue:C-Device
- R17: value 33 -> 1k; symbol Device:R -> OtterIronProRedesign-rescue:R-Device
- U8: renamed from U7; symbol Sensor_Temperature:MCP9700AT-ETT -> OtterIronProRedesign-rescue:MCP9700AT-ETT-Sensor_Temperature
Connections:
- net labels added: +3.3VA, GNDA, ThermoCoupleInput+, ThermoCoupleInput-
- net labels removed: GND, ThermoCoupleInput, V+
- wire segments 24 -> 40
Other:
- note added: "Alternate parts:\nTexas Instruments LMC6482\nAnalog Devices AD8629"
- note added: "JBC C245 Thermocouple:\n1.65mV @100°C\n-0.3mV @0°C\n=> 1.95mV/100°C = 19.5µV/°C\n=>8.5mV @ 450°C"
- note added: "operational amplifiers with higher slew rates need less settling time after\nheater was active before temperature measurement can be taken."
- note added: "positive input is connected to GND close to the connector"
- note removed: "Alternate parts:\nTexas Instruments LMV721IDBVR\nON Semiconductor NCS2003SN2T1G"
- moved on the sheet: C27, C30, R17
