File: ECAD/CurrentSensing.sch (KiCad schematic (older format))
At the start: 6 parts

Commit message: routing almost done
Parts:
- added R21: 1k, Resistor_SMD:R_0402_1005Metric, symbol Device:R
- C32: renamed from C?; symbol Device:C -> OtterIronProRedesign-rescue:C-Device
- C33: renamed from C23; value DNP -> 100nF; symbol Device:C -> OtterIronProRedesign-rescue:C-Device
- NT3: renamed from NT11; symbol Device:Net-Tie_2 -> OtterIronProRedesign-rescue:Net-Tie_2-Device
- NT4: renamed from NT12; symbol Device:Net-Tie_2 -> OtterIronProRedesign-rescue:Net-Tie_2-Device
- R22: renamed from R18; symbol Device:R -> OtterIronProRedesign-rescue:R-Device
- U9: renamed from U?; symbol Amplifier_Current:INA194 -> OtterIronProRedesign-rescue:INA194-Amplifier_Current
Connections:
- net CurrentMeasurement: now also R21.2; no longer U9.1
- net Current+ renamed CurrentIn
- net Current- renamed CurrentOut
- net GND renamed GNDA
- net V+ renamed +3.3VA
- new net: R21.1, U9.1
Other:
- note added: "1.6kHz low pass filter to attenuate PWM frequency"
- moved on the sheet: C32, C33
Changed lines of the file:
@@
 $EndDescr
 $Comp
-L Device:R R18
+L OtterIronProRedesign-rescue:R-Device R22
 U 1 1 5FAB03B5
 P 5000 3250
-F 0 "R18" H 5070 3296 50  0000 L CNN
+F 0 "R22" H 5070 3296 50  0000 L CNN
 F 1 "8m ±1% 2W ±100ppm/°C" H 5070 3205 50  0000 L CNN
 F 2 "Resistor_SMD:R_2512_6332Metric" V 4930 3250 50  0001 C CNN
@@
 $EndComp
 $Comp
-L Device:Net-Tie_2 NT11
+L OtterIronProRedesign-rescue:Net-Tie_2-Device NT3
 U 1 1 5FAB0E9B
 P 4600 3100
-F 0 "NT11" H 4600 3281 50  0000 C CNN
+F 0 "NT3" H 4600 3281 50  0000 C CNN
 F 1 "Net-Tie_2" H 4600 3190 50  0000 C CNN
 F 2 "NetTie:NetTie-2_SMD_Pad0.5mm" H 4600 3100 50  0001 C CNN
@@
 $EndComp
 $Comp
-L Device:Net-Tie_2 NT12
+L OtterIronProRedesign-rescue:Net-Tie_2-Device NT4
 U 1 1 5FAB193B
 P 4600 3400
-F 0 "NT12" H 4600 3581 50  0000 C CNN
+F 0 "NT4" H 4600 3581 50  0000 C CNN
 F 1 "Net-Tie_2" H 4600 3490 50  0000 C CNN
 F 2 "NetTie:NetTie-2_SMD_Pad0.5mm" H 4600 3400 50  0001 C CNN
@@
 Text Notes 5100 3100 0    50   ~ 0
 power dissipation @ nominal current (7.5A): 0.45W
-Text HLabel 2500 3250 0    50   Output ~ 0
+Text HLabel 2200 3250 0    50   Output ~ 0
 CurrentMeasurement
-Text HLabel 2500 2500 0    50   Output ~ 0
-V+
-Text HLabel 2500 3650 0    50   UnSpc ~ 0
-GND
-Wire Wire Line
-	4000 3650 4000 3550
 Text HLabel 5000 2500 1    50   Input ~ 0
-Current+
+CurrentIn
 Text HLabel 5000 4000 3    50   Output ~ 0
-Current-
+CurrentOut
 $Comp
-L Device:C C23
+L OtterIronProRedesign-rescue:C-Device C33
 U 1 1 5FAB674D
-P 2800 3400
-F 0 "C23" H 2915 3446 50  0000 L CNN
-F 1 "DNP" H 2915 3355 50  0000 L CNN
-F 2 "Capacitor_SMD:C_0402_1005Metric" H 2838 3250 50  0001 C CNN
-F 3 "~" H 2800 3400 50  0001 C CNN
-	1    2800 3400
+P 2500 3400
+F 0 "C33" H 2615 3446 50  0000 L CNN
+F 1 "100nF" H 2615 3355 50  0000 L CNN
+F 2 "Capacitor_SMD:C_0402_1005Metric" H 2538 3250 50  0001 C CNN
+F 3 "~" H 2500 3400 50  0001 C CNN
+	1    2500 3400
 	1    0    0    -1
 $EndComp
 Wire Wire Line
-	2500 3250 2800 3250
-Wire Wire Line
-	2800 3250 3600 3250
-Connection ~ 2800 3250
-Wire Wire Line
-	2500 3650 2800 3650
-Wire Wire Line
-	2800 3550 2800 3650
-Connection ~ 2800 3650
-Wire Wire Line
-	2800 3650 4000 3650
+	2200 3250 2500 3250
 Text Notes 7500 3500 0    50   ~ 0
 adjust current sense resistor and amplifier as following:\n3A (standard USB-C PD supplies): 40m ohm + INA193\n5A (some USB-C PD supplies): 25m ohm + INA193\n7A (e.g. bench power supply): 8m ohm + INA194\n\nResistor and amplifier have the same footprint and\ncan be used without changing the layout
 $Comp
-L Amplifier_Current:INA194 U?
+L OtterIronProRedesign-rescue:INA194-Amplifier_Current U9
 U 1 1 5FAE7FB1
 P 3900 3250
-F 0 "U?" H 3900 3731 50  0000 C CNN
+F 0 "U9" H 3900 3731 50  0000 C CNN
 F 1 "INA194" H 3900 3640 50  0000 C CNN
 F 2 "Package_TO_SOT_SMD:SOT-23-5" H 3900 3250 50  0001 C CNN
@@
 $EndComp
 $Comp
-L Device:C C?
+L OtterIronProRedesign-rescue:C-Device C32
 U 1 1 5FAE9929
-P 4250 2650
-F 0 "C?" H 4365 2696 50  0000 L CNN
-F 1 "100nF" H 4365 2605 50  0000 L CNN
-F 2 "Capacitor_SMD:C_0402_1005Metric" H 4288 2500 50  0001 C CNN
-F 3 "~" H 4250 2650 50  0001 C CNN
-	1    4250 2650
+P 4500 2350
+F 0 "C32" H 4615 2396 50  0000 L CNN
+F 1 "100nF" H 4615 2305 50  0000 L CNN
+F 2 "Capacitor_SMD:C_0402_1005Metric" H 4538 2200 50  0001 C CNN
+F 3 "~" H 4500 2350 50  0001 C CNN
+	1    4500 2350
+	1    0    0    -1
+$EndComp
+$Comp
+L power:+3.3VA #PWR084
+U 1 1 5FB0E2B2
+P 4000 2000
+F 0 "#PWR084" H 4000 1850 50  0001 C CNN
+F 1 "+3.3VA" H 4015 2173 50  0000 C CNN
+F 2 "" H 4000 2000 50  0001 C CNN
+F 3 "" H 4000 2000 50  0001 C CNN
+	1    4000 2000
+	1    0    0    -1
+$EndComp
+$Comp
+L power:GNDA #PWR085
+U 1 1 5FB0FBBA
+P 4500 2600
+F 0 "#PWR085" H 4500 2350 50  0001 C CNN
+F 1 "GNDA" H 4505 2427 50  0000 C CNN
+F 2 "" H 4500 2600 50  0001 C CNN
+F 3 "" H 4500 2600 50  0001 C CNN
+	1    4500 2600
 	1    0    0    -1
 $EndComp
 Wire Wire Line
-	2500 2500 4000 2500
+	4000 2000 4000 2100
 Wire Wire Line
-	4000 2500 4000 2950
+	4500 2600 4500 2500
 Wire Wire Line
-	4250 2500 4000 2500
-Connection ~ 4000 2500
-Text HLabel 4250 2900 3    50   UnSpc ~ 0
-GND
+	4500 2200 4500 2100
 Wire Wire Line
-	4250 2800 4250 2900
+	4500 2100 4000 2100
+Connection ~ 4000 2100
+Wire Wire Line
+	4000 2100 4000 2950
+$Comp
+L power:GNDA #PWR087
+U 1 1 5FB1209A
+P 4000 3750
+F 0 "#PWR087" H 4000 3500 50  0001 C CNN
+F 1 "GNDA" H 4005 3577 50  0000 C CNN
+F 2 "" H 4000 3750 50  0001 C CNN
+F 3 "" H 4000 3750 50  0001 C CNN
+	1    4000 3750
+	1    0    0    -1
+$EndComp
+$Comp
+L power:GNDA #PWR086
+U 1 1 5FB1235D
+P 2500 3750
+F 0 "#PWR086" H 2500 3500 50  0001 C CNN
+F 1 "GNDA" H 2505 3577 50  0000 C CNN
+F 2 "" H 2500 3750 50  0001 C CNN
+F 3 "" H 2500 3750 50  0001 C CNN
+	1    2500 3750
+	1    0    0    -1
+$EndComp
+Wire Wire Line
+	2500 3550 2500 3750
+Wire Wire Line
+	4000 3550 4000 3750
+$Comp
+L Device:R R21
+U 1 1 5FB1C215
+P 3250 3250
+F 0 "R21" V 3043 3250 50  0000 C CNN
+F 1 "1k" V 3134 3250 50  0000 C CNN
+F 2 "Resistor_SMD:R_0402_1005Metric" V 3180 3250 50  0001 C CNN
+F 3 "~" H 3250 3250 50  0001 C CNN
+	1    3250 3250
+	0    1    1    0
+$EndComp
+Wire Wire Line
+	3100 3250 2500 3250
+Connection ~ 2500 3250
+Wire Wire Line
+	3400 3250 3600 3250
+Text Notes 2000 3000 0    50   ~ 0
+1.6kHz low pass filter to attenuate PWM frequency
 $EndSCHEMATC

Commit message: swapped microcontroller
Parts:
- NT3, NT4: footprint NetTie:NetTie-2_SMD_Pad0.5mm -> ECAD:NetTie-2_SMD_Pad0.25mm
Changed lines of the file:
@@
 $Descr A4 11693 8268
 encoding utf-8
-Sheet 8 8
+Sheet 7 8
 Title ""
 Date ""
@@
 F 0 "NT3" H 4600 3281 50  0000 C CNN
 F 1 "Net-Tie_2" H 4600 3190 50  0000 C CNN
-F 2 "NetTie:NetTie-2_SMD_Pad0.5mm" H 4600 3100 50  0001 C CNN
+F 2 "ECAD:NetTie-2_SMD_Pad0.25mm" H 4600 3100 50  0001 C CNN
 F 3 "~" H 4600 3100 50  0001 C CNN
 	1    4600 3100
@@
 F 0 "NT4" H 4600 3581 50  0000 C CNN
 F 1 "Net-Tie_2" H 4600 3490 50  0000 C CNN
-F 2 "NetTie:NetTie-2_SMD_Pad0.5mm" H 4600 3400 50  0001 C CNN
+F 2 "ECAD:NetTie-2_SMD_Pad0.25mm" H 4600 3400 50  0001 C CNN
 F 3 "~" H 4600 3400 50  0001 C CNN
 	1    4600 3400

Commit message: more routing + some component changes
Parts:
- R16: renamed from R22; value 8m ±1% 2W ±100ppm/°C -> 4m ±1% 2W ±100ppm/°C; LCSC C459682 -> C76237; manf# RLP25FEGR015 -> MRF6432(2512)LR004FTS
- U7: renamed from U9; value INA194 -> INA195; LCSC C37807 -> C34542; manf# INA194AIDBVR -> INA195AIDBVR
- renumbered C33 to C24, C32 to C25, R21 to R15
Other:
- note added: "power dissipation @ nominal current (7.5A): 0.225W"
- note removed: "power dissipation @ nominal current (7.5A): 0.45W"
Changed lines of the file:
@@
 $EndDescr
 $Comp
-L OtterIronProRedesign-rescue:R-Device R22
+L OtterIronProRedesign-rescue:R-Device R16
 U 1 1 5FAB03B5
 P 5000 3250
-F 0 "R22" H 5070 3296 50  0000 L CNN
-F 1 "8m ±1% 2W ±100ppm/°C" H 5070 3205 50  0000 L CNN
+F 0 "R16" H 5070 3296 50  0000 L CNN
+F 1 "4m ±1% 2W ±100ppm/°C" H 5070 3205 50  0000 L CNN
 F 2 "Resistor_SMD:R_2512_6332Metric" V 4930 3250 50  0001 C CNN
 F 3 "~" H 5000 3250 50  0001 C CNN
-F 4 "RLP25FEGR015" H 5000 3250 50  0001 C CNN "manf#"
-F 5 "C459682" H 5000 3250 50  0001 C CNN "LCSC"
+F 4 "MRF6432(2512)LR004FTS" H 5000 3250 50  0001 C CNN "manf#"
+F 5 "C76237" H 5000 3250 50  0001 C CNN "LCSC"
 	1    5000 3250
 	1    0    0    -1
@@
 use kelvin connections
 Text Notes 5100 3100 0    50   ~ 0
-power dissipation @ nominal current (7.5A): 0.45W
+power dissipation @ nominal current (7.5A): 0.225W
 Text HLabel 2200 3250 0    50   Output ~ 0
 CurrentMeasurement
@@
 CurrentOut
 $Comp
-L OtterIronProRedesign-rescue:C-Device C33
+L OtterIronProRedesign-rescue:C-Device C24
 U 1 1 5FAB674D
 P 2500 3400
-F 0 "C33" H 2615 3446 50  0000 L CNN
+F 0 "C24" H 2615 3446 50  0000 L CNN
 F 1 "100nF" H 2615 3355 50  0000 L CNN
 F 2 "Capacitor_SMD:C_0402_1005Metric" H 2538 3250 50  0001 C CNN
@@
 adjust current sense resistor and amplifier as following:\n3A (standard USB-C PD supplies): 40m ohm + INA193\n5A (some USB-C PD supplies): 25m ohm + INA193\n7A (e.g. bench power supply): 8m ohm + INA194\n\nResistor and amplifier have the same footprint and\ncan be used without changing the layout
 $Comp
-L OtterIronProRedesign-rescue:INA194-Amplifier_Current U9
+L OtterIronProRedesign-rescue:INA194-Amplifier_Current U7
 U 1 1 5FAE7FB1
 P 3900 3250
-F 0 "U9" H 3900 3731 50  0000 C CNN
-F 1 "INA194" H 3900 3640 50  0000 C CNN
+F 0 "U7" H 3900 3731 50  0000 C CNN
+F 1 "INA195" H 3900 3640 50  0000 C CNN
 F 2 "Package_TO_SOT_SMD:SOT-23-5" H 3900 3250 50  0001 C CNN
 F 3 "http://www.ti.com/lit/ds/symlink/ina193.pdf" H 3900 3250 50  0001 C CNN
-F 4 "INA194AIDBVR" H 3900 3250 50  0001 C CNN "manf#"
-F 5 "C37807" H 3900 3250 50  0001 C CNN "LCSC"
+F 4 "INA195AIDBVR" H 3900 3250 50  0001 C CNN "manf#"
+F 5 "C34542" H 3900 3250 50  0001 C CNN "LCSC"
 	1    3900 3250
 	-1   0    0    -1
 $EndComp
 $Comp
-L OtterIronProRedesign-rescue:C-Device C32
+L OtterIronProRedesign-rescue:C-Device C25
 U 1 1 5FAE9929
 P 4500 2350
-F 0 "C32" H 4615 2396 50  0000 L CNN
+F 0 "C25" H 4615 2396 50  0000 L CNN
 F 1 "100nF" H 4615 2305 50  0000 L CNN
 F 2 "Capacitor_SMD:C_0402_1005Metric" H 4538 2200 50  0001 C CNN
@@
 $EndComp
 $Comp
-L power:+3.3VA #PWR084
+L power:+3.3VA #PWR076
 U 1 1 5FB0E2B2
 P 4000 2000
-F 0 "#PWR084" H 4000 1850 50  0001 C CNN
+F 0 "#PWR076" H 4000 1850 50  0001 C CNN
 F 1 "+3.3VA" H 4015 2173 50  0000 C CNN
 F 2 "" H 4000 2000 50  0001 C CNN
@@
 $EndComp
 $Comp
-L power:GNDA #PWR085
+L power:GNDA #PWR078
 U 1 1 5FB0FBBA
 P 4500 2600
-F 0 "#PWR085" H 4500 2350 50  0001 C CNN
+F 0 "#PWR078" H 4500 2350 50  0001 C CNN
 F 1 "GNDA" H 4505 2427 50  0000 C CNN
 F 2 "" H 4500 2600 50  0001 C CNN
@@
 	4000 2100 4000 2950
 $Comp
-L power:GNDA #PWR087
+L power:GNDA #PWR077
 U 1 1 5FB1209A
 P 4000 3750
-F 0 "#PWR087" H 4000 3500 50  0001 C CNN
+F 0 "#PWR077" H 4000 3500 50  0001 C CNN
 F 1 "GNDA" H 4005 3577 50  0000 C CNN
 F 2 "" H 4000 3750 50  0001 C CNN
@@
 $EndComp
 $Comp
-L power:GNDA #PWR086
+L power:GNDA #PWR075
 U 1 1 5FB1235D
 P 2500 3750
-F 0 "#PWR086" H 2500 3500 50  0001 C CNN
+F 0 "#PWR075" H 2500 3500 50  0001 C CNN
 F 1 "GNDA" H 2505 3577 50  0000 C CNN
 F 2 "" H 2500 3750 50  0001 C CNN
@@
 	4000 3550 4000 3750
 $Comp
-L Device:R R21
+L Device:R R15
 U 1 1 5FB1C215
 P 3250 3250
-F 0 "R21" V 3043 3250 50  0000 C CNN
+F 0 "R15" V 3043 3250 50  0000 C CNN
 F 1 "1k" V 3134 3250 50  0000 C CNN
 F 2 "Resistor_SMD:R_0402_1005Metric" V 3180 3250 50  0001 C CNN
