File: ECAD/InputFilter.sch (KiCad schematic (older format))
At the start: 4 parts

Commit message: more routing + some component changes
Parts:
- C28: renamed from C36; LCSC (none) -> C134808; manf# (none) -> VZH101M1HTR-1010
- L1: LCSC (none) -> C149568; manf# (none) -> MWSA1205-1R0MT
- renumbered C34 to C26, C35 to C27
Changed lines of the file:
@@
 P 4400 3750
 AR Path="/5FA8950E/5FB22198" Ref="C?"  Part="1"
-AR Path="/5FB20F90/5FB22198" Ref="C34"  Part="1"
-F 0 "C34" H 4515 3796 50  0000 L CNN
+AR Path="/5FB20F90/5FB22198" Ref="C26"  Part="1"
+F 0 "C26" H 4515 3796 50  0000 L CNN
 F 1 "1µF 35V" H 4515 3705 50  0000 L CNN
 F 2 "Capacitor_SMD:C_0402_1005Metric" H 4438 3600 50  0001 C CNN
@@
 P 5000 3750
 AR Path="/5FA8950E/5FB2219E" Ref="C?"  Part="1"
-AR Path="/5FB20F90/5FB2219E" Ref="C35"  Part="1"
-F 0 "C35" H 5115 3796 50  0000 L CNN
+AR Path="/5FB20F90/5FB2219E" Ref="C27"  Part="1"
+F 0 "C27" H 5115 3796 50  0000 L CNN
 F 1 "1µF 35V" H 5115 3705 50  0000 L CNN
 F 2 "Capacitor_SMD:C_0402_1005Metric" H 5038 3600 50  0001 C CNN
@@
 P 5600 3750
 AR Path="/5FA8950E/5FB221AA" Ref="C?"  Part="1"
-AR Path="/5FB20F90/5FB221AA" Ref="C36"  Part="1"
-F 0 "C36" H 5718 3796 50  0000 L CNN
+AR Path="/5FB20F90/5FB221AA" Ref="C28"  Part="1"
+F 0 "C28" H 5718 3796 50  0000 L CNN
 F 1 "100µF 35V" H 5718 3705 50  0000 L CNN
 F 2 "Capacitor_SMD:CP_Elec_10x10.5" H 5638 3600 50  0001 C CNN
 F 3 "~" H 5600 3750 50  0001 C CNN
+F 4 "VZH101M1HTR-1010" H 5600 3750 50  0001 C CNN "manf#"
+F 5 "C134808" H 5600 3750 50  0001 C CNN "LCSC"
 	1    5600 3750
 	1    0    0    -1
@@
 P 5000 4000
 AR Path="/5FA8950E/5FB221B7" Ref="#PWR?"  Part="1"
-AR Path="/5FB20F90/5FB221B7" Ref="#PWR088"  Part="1"
-F 0 "#PWR088" H 5000 3750 50  0001 C CNN
+AR Path="/5FB20F90/5FB221B7" Ref="#PWR079"  Part="1"
+F 0 "#PWR079" H 5000 3750 50  0001 C CNN
 F 1 "GND" H 5005 3827 50  0000 C CNN
 F 2 "" H 5000 4000 50  0001 C CNN
@@
 F 2 "Inductor_SMD:L_12x12mm_H8mm" H 5000 3250 50  0001 C CNN
 F 3 "~" H 5000 3250 50  0001 C CNN
+F 4 "MWSA1205-1R0MT" V 5000 3250 50  0001 C CNN "manf#"
+F 5 "C149568" V 5000 3250 50  0001 C CNN "LCSC"
 	1    5000 3250
 	1    0    0    -1
