File: ECAD/USB.sch (KiCad schematic (older format))
At the start: 10 parts, among them J6 USB_C_Receptacle_USB2.0, U3 USBLC6-4SC6, U4 STUSB4500QTR

Commit message: routing almost done
Parts:
- removed D2: 22V 10A, Diode_SMD:D_SMB, symbol Device:D_Zener
- C13: renamed from C11; symbol Device:C -> OtterIronProRedesign-rescue:C-Device
- C14: renamed from C12; symbol Device:C -> OtterIronProRedesign-rescue:C-Device
- C15: renamed from C9; symbol Device:C -> OtterIronProRedesign-rescue:C-Device
- C16: renamed from C10; symbol Device:C -> OtterIronProRedesign-rescue:C-Device
- J25: renamed from J6; symbol Connector:USB_C_Receptacle_USB2.0 -> OtterIronProRedesign-rescue:USB_C_Receptacle_USB2.0-Connector
- R10: renamed from R9; symbol Device:R -> OtterIronProRedesign-rescue:R-Device
- R11: renamed from R10; symbol Device:R -> OtterIronProRedesign-rescue:R-Device
- U2: renamed from U4; symbol Interface_USB:STUSB4500QTR -> OtterIronProRedesign-rescue:STUSB4500QTR-Interface_USB
- U3: symbol Power_Protection:USBLC6-4SC6 -> OtterIronProRedesign-rescue:USBLC6-4SC6-Power_Protection
Connections:
- net CC1: now also U3.3 (I/O2); no longer U3.1 (I/O1)
- net CC2: now also U3.1 (I/O1); no longer U3.3 (I/O2)
Changed lines of the file:
@@
 $EndDescr
 $Comp
-L Connector:USB_C_Receptacle_USB2.0 J6
+L OtterIronProRedesign-rescue:USB_C_Receptacle_USB2.0-Connector J25
 U 1 1 5FA49D2A
 P 1900 3700
-F 0 "J6" H 2007 4567 50  0000 C CNN
+F 0 "J25" H 2007 4567 50  0000 C CNN
 F 1 "USB_C_Receptacle_USB2.0" H 2007 4476 50  0000 C CNN
 F 2 "Connector_USB:USB_C_Receptacle_XKB_U262-16XN-4BVC11" H 2050 3700 50  0001 C CNN
@@
 $EndComp
 $Comp
-L Interface_USB:STUSB4500QTR U4
+L OtterIronProRedesign-rescue:STUSB4500QTR-Interface_USB U2
 U 1 1 5FA4BD0C
 P 5350 3800
-F 0 "U4" H 5350 2811 50  0000 C CNN
+F 0 "U2" H 5350 2811 50  0000 C CNN
 F 1 "STUSB4500QTR" H 5350 2720 50  0000 C CNN
 F 2 "Package_DFN_QFN:QFN-24-1EP_4x4mm_P0.5mm_EP2.7x2.7mm" H 5350 3800 50  0001 C CNN
@@
 $EndComp
 $Comp
-L Power_Protection:USBLC6-4SC6 U3
+L OtterIronProRedesign-rescue:USBLC6-4SC6-Power_Protection U3
 U 1 1 5FA4C613
 P 3350 5400
@@
 $EndComp
 $Comp
-L Device:C C9
+L OtterIronProRedesign-rescue:C-Device C15
 U 1 1 5FA4F263
 P 3000 2850
-F 0 "C9" H 3115 2896 50  0000 L CNN
+F 0 "C15" H 3115 2896 50  0000 L CNN
 F 1 "100nF" H 3115 2805 50  0000 L CNN
 F 2 "Capacitor_SMD:C_0402_1005Metric" H 3038 2700 50  0001 C CNN
@@
 $EndComp
 $Comp
-L Device:C C11
+L OtterIronProRedesign-rescue:C-Device C13
 U 1 1 5FA4F950
 P 5900 2350
-F 0 "C11" V 5648 2350 50  0000 C CNN
+F 0 "C13" V 5648 2350 50  0000 C CNN
 F 1 "1µF 35V" V 5739 2350 50  0000 C CNN
 F 2 "Capacitor_SMD:C_0402_1005Metric" H 5938 2200 50  0001 C CNN
@@
 	2600 3600 3050 3600
 $Comp
-L power:GND #PWR046
+L OtterIronProRedesign-rescue:GND-power #PWR051
 U 1 1 5FA54DF1
 P 4650 4600
-F 0 "#PWR046" H 4650 4350 50  0001 C CNN
+F 0 "#PWR051" H 4650 4350 50  0001 C CNN
 F 1 "GND" H 4655 4427 50  0000 C CNN
 F 2 "" H 4650 4600 50  0001 C CNN
@@
 NoConn ~ 5950 4400
 $Comp
-L power:GND #PWR038
+L OtterIronProRedesign-rescue:GND-power #PWR049
 U 1 1 5FA58BC0
 P 1600 4600
-F 0 "#PWR038" H 1600 4350 50  0001 C CNN
+F 0 "#PWR049" H 1600 4350 50  0001 C CNN
 F 1 "GND" H 1605 4427 50  0000 C CNN
 F 2 "" H 1600 4600 50  0001 C CNN
@@
 $EndComp
 $Comp
-L power:GND #PWR039
+L OtterIronProRedesign-rescue:GND-power #PWR050
 U 1 1 5FA58FBE
 P 1900 4600
-F 0 "#PWR039" H 1900 4350 50  0001 C CNN
+F 0 "#PWR050" H 1900 4350 50  0001 C CNN
 F 1 "GND" H 1905 4427 50  0000 C CNN
 F 2 "" H 1900 4600 50  0001 C CNN
@@
 	2500 3100 2600 3100
 $Comp
-L power:GND #PWR040
+L OtterIronProRedesign-rescue:GND-power #PWR047
 U 1 1 5FA5C044
 P 3000 3000
-F 0 "#PWR040" H 3000 2750 50  0001 C CNN
+F 0 "#PWR047" H 3000 2750 50  0001 C CNN
 F 1 "GND" H 3005 2827 50  0000 C CNN
 F 2 "" H 3000 3000 50  0001 C CNN
@@
 $EndComp
 $Comp
-L power:+3.3V #PWR047
+L OtterIronProRedesign-rescue:+3.3V-power #PWR045
 U 1 1 5FA5D1A6
 P 5350 2900
-F 0 "#PWR047" H 5350 2750 50  0001 C CNN
+F 0 "#PWR045" H 5350 2750 50  0001 C CNN
 F 1 "+3.3V" H 5365 3073 50  0000 C CNN
 F 2 "" H 5350 2900 50  0001 C CNN
@@
 $EndComp
 $Comp
-L Device:C C12
+L OtterIronProRedesign-rescue:C-Device C14
 U 1 1 5FA65417
 P 5900 2800
-F 0 "C12" V 5648 2800 50  0000 C CNN
+F 0 "C14" V 5648 2800 50  0000 C CNN
 F 1 "1µF 35V" V 5739 2800 50  0000 C CNN
 F 2 "Capacitor_SMD:C_0402_1005Metric" H 5938 2650 50  0001 C CNN
@@
 	6150 2800 6150 2900
 $Comp
-L power:GND #PWR049
+L OtterIronProRedesign-rescue:GND-power #PWR046
 U 1 1 5FA74B1E
 P 6150 2900
-F 0 "#PWR049" H 6150 2650 50  0001 C CNN
+F 0 "#PWR046" H 6150 2650 50  0001 C CNN
 F 1 "GND" H 6155 2727 50  0000 C CNN
 F 2 "" H 6150 2900 50  0001 C CNN
@@
 	4750 4300 4650 4300
 $Comp
-L Device:R R10
+L OtterIronProRedesign-rescue:R-Device R11
 U 1 1 5FA787AB
 P 4500 3900
-F 0 "R10" V 4293 3900 50  0000 C CNN
+F 0 "R11" V 4293 3900 50  0000 C CNN
 F 1 "10k" V 4384 3900 50  0000 C CNN
 F 2 "Resistor_SMD:R_0402_1005Metric" V 4430 3900 50  0001 C CNN
@@
 NoConn ~ 5950 3900
 $Comp
-L power:GND #PWR048
+L OtterIronProRedesign-rescue:GND-power #PWR053
 U 1 1 5FA7B10B
 P 5350 5000
-F 0 "#PWR048" H 5350 4750 50  0001 C CNN
+F 0 "#PWR053" H 5350 4750 50  0001 C CNN
 F 1 "GND" H 5355 4827 50  0000 C CNN
 F 2 "" H 5350 5000 50  0001 C CNN
@@
 	2950 5500 2850 5500
 Text Label 2850 5300 2    50   ~ 0
+CC2
+Text Label 2850 5500 2    50   ~ 0
 CC1
-Text Label 2850 5500 2    50   ~ 0
-CC2
 Text Label 3850 5500 0    50   ~ 0
 USB_P
@@
 USB_N
 $Comp
-L power:+3.3V #PWR041
+L OtterIronProRedesign-rescue:+3.3V-power #PWR052
 U 1 1 5FA81F4A
 P 3350 4750
-F 0 "#PWR041" H 3350 4600 50  0001 C CNN
+F 0 "#PWR052" H 3350 4600 50  0001 C CNN
 F 1 "+3.3V" H 3365 4923 50  0000 C CNN
 F 2 "" H 3350 4750 50  0001 C CNN
@@
 $EndComp
 $Comp
-L power:GND #PWR042
+L OtterIronProRedesign-rescue:GND-power #PWR054
 U 1 1 5FA8260F
 P 3350 5800
-F 0 "#PWR042" H 3350 5550 50  0001 C CNN
+F 0 "#PWR054" H 3350 5550 50  0001 C CNN
 F 1 "GND" H 3355 5627 50  0000 C CNN
 F 2 "" H 3350 5800 50  0001 C CNN
@@
 	3350 5000 3350 4750
 $Comp
-L Device:R R9
+L OtterIronProRedesign-rescue:R-Device R10
 U 1 1 5FA85F86
 P 4500 3100
-F 0 "R9" V 4293 3100 50  0000 C CNN
+F 0 "R10" V 4293 3100 50  0000 C CNN
 F 1 "10k" V 4384 3100 50  0000 C CNN
 F 2 "Resistor_SMD:R_0402_1005Metric" V 4430 3100 50  0001 C CNN
@@
 	0    1    1    0
 $EndComp
-$Comp
-L power:GND #PWR045
-U 1 1 5FA86339
-P 4200 3150
-F 0 "#PWR045" H 4200 2900 50  0001 C CNN
-F 1 "GND" H 4205 2977 50  0000 C CNN
-F 2 "" H 4200 3150 50  0001 C CNN
-F 3 "" H 4200 3150 50  0001 C CNN
-	1    4200 3150
-	1    0    0    -1
-$EndComp
 Wire Wire Line
 	4200 3150 4200 3100
@@
 	5950 3700 6050 3700
 $Comp
-L Device:C C10
+L OtterIronProRedesign-rescue:C-Device C16
 U 1 1 5FA82628
 P 3500 2850
-F 0 "C10" H 3615 2896 50  0000 L CNN
+F 0 "C16" H 3615 2896 50  0000 L CNN
 F 1 "1µF 35V" H 3615 2805 50  0000 L CNN
 F 2 "Capacitor_SMD:C_0402_1005Metric" H 3538 2700 50  0001 C CNN
@@
 $EndComp
 $Comp
-L power:GND #PWR043
+L OtterIronProRedesign-rescue:GND-power #PWR048
 U 1 1 5FA82F20
 P 3500 3000
-F 0 "#PWR043" H 3500 2750 50  0001 C CNN
+F 0 "#PWR048" H 3500 2750 50  0001 C CNN
 F 1 "GND" H 3505 2827 50  0000 C CNN
 F 2 "" H 3500 3000 50  0001 C CNN
@@
 Text Label 4250 3900 2    50   ~ 0
 VBusIn
-$Comp
-L Device:D_Zener D?
-U 1 1 5FAA198D
-P 4050 2900
-AR Path="/5FAA198D" Ref="D?"  Part="1"
-AR Path="/5FA49B46/5FAA198D" Ref="D2"  Part="1"
-F 0 "D2" V 4004 2980 50  0000 L CNN
-F 1 "22V 10A" V 4095 2980 50  0000 L CNN
-F 2 "Diode_SMD:D_SMB" H 4050 2900 50  0001 C CNN
-F 3 "~" H 4050 2900 50  0001 C CNN
-F 4 "SMBJ22A" V 4050 2900 50  0001 C CNN "manf#"
-F 5 "C224015" V 4050 2900 50  0001 C CNN "LCSC"
-	1    4050 2900
-	0    1    1    0
-$EndComp
-Wire Wire Line
-	3500 2700 4050 2700
-Wire Wire Line
-	4050 2750 4050 2700
-Connection ~ 4050 2700
-Wire Wire Line
-	4050 2700 4300 2700
-$Comp
-L power:GND #PWR044
-U 1 1 5FAA4642
-P 4050 3050
-F 0 "#PWR044" H 4050 2800 50  0001 C CNN
-F 1 "GND" H 4055 2877 50  0000 C CNN
-F 2 "" H 4050 3050 50  0001 C CNN
-F 3 "" H 4050 3050 50  0001 C CNN
-	1    4050 3050
-	1    0    0    -1
-$EndComp
+Wire Wire Line
+	3500 2700 4300 2700
+$Comp
+L OtterIronProRedesign-rescue:GND-power #PWR0101
+U 1 1 5FC21147
+P 4200 3150
+F 0 "#PWR0101" H 4200 2900 50  0001 C CNN
+F 1 "GND" H 4205 2977 50  0000 C CNN
+F 2 "" H 4200 3150 50  0001 C CNN
+F 3 "" H 4200 3150 50  0001 C CNN
+	1    4200 3150
+	1    0    0    -1
+$EndComp

Commit message: more routing + some component changes
Parts:
- renumbered C15 to C12, C16 to C13, C13 to C14, C14 to C15, J25 to J19, U3 to U2, U2 to U3
Changed lines of the file:
@@
 $EndDescr
 $Comp
-L OtterIronProRedesign-rescue:USB_C_Receptacle_USB2.0-Connector J25
+L OtterIronProRedesign-rescue:USB_C_Receptacle_USB2.0-Connector J19
 U 1 1 5FA49D2A
 P 1900 3700
-F 0 "J25" H 2007 4567 50  0000 C CNN
+F 0 "J19" H 2007 4567 50  0000 C CNN
 F 1 "USB_C_Receptacle_USB2.0" H 2007 4476 50  0000 C CNN
 F 2 "Connector_USB:USB_C_Receptacle_XKB_U262-16XN-4BVC11" H 2050 3700 50  0001 C CNN
@@
 $EndComp
 $Comp
-L OtterIronProRedesign-rescue:STUSB4500QTR-Interface_USB U2
+L OtterIronProRedesign-rescue:STUSB4500QTR-Interface_USB U3
 U 1 1 5FA4BD0C
 P 5350 3800
-F 0 "U2" H 5350 2811 50  0000 C CNN
+F 0 "U3" H 5350 2811 50  0000 C CNN
 F 1 "STUSB4500QTR" H 5350 2720 50  0000 C CNN
 F 2 "Package_DFN_QFN:QFN-24-1EP_4x4mm_P0.5mm_EP2.7x2.7mm" H 5350 3800 50  0001 C CNN
@@
 $EndComp
 $Comp
-L OtterIronProRedesign-rescue:USBLC6-4SC6-Power_Protection U3
+L OtterIronProRedesign-rescue:USBLC6-4SC6-Power_Protection U2
 U 1 1 5FA4C613
 P 3350 5400
-F 0 "U3" H 3350 5981 50  0000 C CNN
+F 0 "U2" H 3350 5981 50  0000 C CNN
 F 1 "USBLC6-4SC6" H 3350 5890 50  0000 C CNN
 F 2 "Package_TO_SOT_SMD:SOT-23-6" H 3350 4900 50  0001 C CNN
@@
 $EndComp
 $Comp
-L OtterIronProRedesign-rescue:C-Device C15
+L OtterIronProRedesign-rescue:C-Device C12
 U 1 1 5FA4F263
 P 3000 2850
-F 0 "C15" H 3115 2896 50  0000 L CNN
+F 0 "C12" H 3115 2896 50  0000 L CNN
 F 1 "100nF" H 3115 2805 50  0000 L CNN
 F 2 "Capacitor_SMD:C_0402_1005Metric" H 3038 2700 50  0001 C CNN
@@
 $EndComp
 $Comp
-L OtterIronProRedesign-rescue:C-Device C13
+L OtterIronProRedesign-rescue:C-Device C14
 U 1 1 5FA4F950
 P 5900 2350
-F 0 "C13" V 5648 2350 50  0000 C CNN
+F 0 "C14" V 5648 2350 50  0000 C CNN
 F 1 "1µF 35V" V 5739 2350 50  0000 C CNN
 F 2 "Capacitor_SMD:C_0402_1005Metric" H 5938 2200 50  0001 C CNN
@@
 	2600 3600 3050 3600
 $Comp
-L OtterIronProRedesign-rescue:GND-power #PWR051
+L OtterIronProRedesign-rescue:GND-power #PWR054
 U 1 1 5FA54DF1
 P 4650 4600
-F 0 "#PWR051" H 4650 4350 50  0001 C CNN
+F 0 "#PWR054" H 4650 4350 50  0001 C CNN
 F 1 "GND" H 4655 4427 50  0000 C CNN
 F 2 "" H 4650 4600 50  0001 C CNN
@@
 NoConn ~ 5950 4400
 $Comp
-L OtterIronProRedesign-rescue:GND-power #PWR049
+L OtterIronProRedesign-rescue:GND-power #PWR047
 U 1 1 5FA58BC0
 P 1600 4600
-F 0 "#PWR049" H 1600 4350 50  0001 C CNN
+F 0 "#PWR047" H 1600 4350 50  0001 C CNN
 F 1 "GND" H 1605 4427 50  0000 C CNN
 F 2 "" H 1600 4600 50  0001 C CNN
@@
 $EndComp
 $Comp
-L OtterIronProRedesign-rescue:GND-power #PWR050
+L OtterIronProRedesign-rescue:GND-power #PWR048
 U 1 1 5FA58FBE
 P 1900 4600
-F 0 "#PWR050" H 1900 4350 50  0001 C CNN
+F 0 "#PWR048" H 1900 4350 50  0001 C CNN
 F 1 "GND" H 1905 4427 50  0000 C CNN
 F 2 "" H 1900 4600 50  0001 C CNN
@@
 	2500 3100 2600 3100
 $Comp
-L OtterIronProRedesign-rescue:GND-power #PWR047
+L OtterIronProRedesign-rescue:GND-power #PWR049
 U 1 1 5FA5C044
 P 3000 3000
-F 0 "#PWR047" H 3000 2750 50  0001 C CNN
+F 0 "#PWR049" H 3000 2750 50  0001 C CNN
 F 1 "GND" H 3005 2827 50  0000 C CNN
 F 2 "" H 3000 3000 50  0001 C CNN
@@
 $EndComp
 $Comp
-L OtterIronProRedesign-rescue:+3.3V-power #PWR045
+L OtterIronProRedesign-rescue:+3.3V-power #PWR055
 U 1 1 5FA5D1A6
 P 5350 2900
-F 0 "#PWR045" H 5350 2750 50  0001 C CNN
+F 0 "#PWR055" H 5350 2750 50  0001 C CNN
 F 1 "+3.3V" H 5365 3073 50  0000 C CNN
 F 2 "" H 5350 2900 50  0001 C CNN
@@
 $EndComp
 $Comp
-L OtterIronProRedesign-rescue:C-Device C14
+L OtterIronProRedesign-rescue:C-Device C15
 U 1 1 5FA65417
 P 5900 2800
-F 0 "C14" V 5648 2800 50  0000 C CNN
+F 0 "C15" V 5648 2800 50  0000 C CNN
 F 1 "1µF 35V" V 5739 2800 50  0000 C CNN
 F 2 "Capacitor_SMD:C_0402_1005Metric" H 5938 2650 50  0001 C CNN
@@
 	6150 2800 6150 2900
 $Comp
-L OtterIronProRedesign-rescue:GND-power #PWR046
+L OtterIronProRedesign-rescue:GND-power #PWR057
 U 1 1 5FA74B1E
 P 6150 2900
-F 0 "#PWR046" H 6150 2650 50  0001 C CNN
+F 0 "#PWR057" H 6150 2650 50  0001 C CNN
 F 1 "GND" H 6155 2727 50  0000 C CNN
 F 2 "" H 6150 2900 50  0001 C CNN
@@
 NoConn ~ 5950 3900
 $Comp
-L OtterIronProRedesign-rescue:GND-power #PWR053
+L OtterIronProRedesign-rescue:GND-power #PWR056
 U 1 1 5FA7B10B
 P 5350 5000
-F 0 "#PWR053" H 5350 4750 50  0001 C CNN
+F 0 "#PWR056" H 5350 4750 50  0001 C CNN
 F 1 "GND" H 5355 4827 50  0000 C CNN
 F 2 "" H 5350 5000 50  0001 C CNN
@@
 USB_N
 $Comp
-L OtterIronProRedesign-rescue:+3.3V-power #PWR052
+L OtterIronProRedesign-rescue:+3.3V-power #PWR050
 U 1 1 5FA81F4A
 P 3350 4750
-F 0 "#PWR052" H 3350 4600 50  0001 C CNN
+F 0 "#PWR050" H 3350 4600 50  0001 C CNN
 F 1 "+3.3V" H 3365 4923 50  0000 C CNN
 F 2 "" H 3350 4750 50  0001 C CNN
@@
 $EndComp
 $Comp
-L OtterIronProRedesign-rescue:GND-power #PWR054
+L OtterIronProRedesign-rescue:GND-power #PWR051
 U 1 1 5FA8260F
 P 3350 5800
-F 0 "#PWR054" H 3350 5550 50  0001 C CNN
+F 0 "#PWR051" H 3350 5550 50  0001 C CNN
 F 1 "GND" H 3355 5627 50  0000 C CNN
 F 2 "" H 3350 5800 50  0001 C CNN
@@
 	5950 3700 6050 3700
 $Comp
-L OtterIronProRedesign-rescue:C-Device C16
+L OtterIronProRedesign-rescue:C-Device C13
 U 1 1 5FA82628
 P 3500 2850
-F 0 "C16" H 3615 2896 50  0000 L CNN
+F 0 "C13" H 3615 2896 50  0000 L CNN
 F 1 "1µF 35V" H 3615 2805 50  0000 L CNN
 F 2 "Capacitor_SMD:C_0402_1005Metric" H 3538 2700 50  0001 C CNN
@@
 $EndComp
 $Comp
-L OtterIronProRedesign-rescue:GND-power #PWR048
+L OtterIronProRedesign-rescue:GND-power #PWR052
 U 1 1 5FA82F20
 P 3500 3000
-F 0 "#PWR048" H 3500 2750 50  0001 C CNN
+F 0 "#PWR052" H 3500 2750 50  0001 C CNN
 F 1 "GND" H 3505 2827 50  0000 C CNN
 F 2 "" H 3500 3000 50  0001 C CNN
@@
 	3500 2700 4300 2700
 $Comp
-L OtterIronProRedesign-rescue:GND-power #PWR0101
+L OtterIronProRedesign-rescue:GND-power #PWR053
 U 1 1 5FC21147
 P 4200 3150
-F 0 "#PWR0101" H 4200 2900 50  0001 C CNN
+F 0 "#PWR053" H 4200 2900 50  0001 C CNN
 F 1 "GND" H 4205 2977 50  0000 C CNN
 F 2 "" H 4200 3150 50  0001 C CNN
